Commit message: New aliengo urdf

File: legged_controllers/config/aliengo/aliengo.urdf (robot description, URDF)
Before this commit: robot aliengo, 19 links, 18 joints
Links:
- link lf_hip: geometry collision cylinder length=0.0418 radius=0.046; visual mesh filename=package://aliengo_description/meshes/hip.dae scale=1 1 1
- link lf_lowerleg: geometry collision box size=0.25 0.0208 0.016; visual mesh filename=package://aliengo_description/meshes/calf.dae scale=1 1 1
- link lf_upperleg: geometry collision box size=0.25 0.0374 0.043; visual mesh filename=package://aliengo_description/meshes/thigh.dae scale=1 1 1
- link lh_hip: geometry collision cylinder length=0.0418 radius=0.046; visual mesh filename=package://aliengo_description/meshes/hip.dae scale=1 1 1
- link lh_lowerleg: geometry collision box size=0.25 0.0208 0.016; visual mesh filename=package://aliengo_description/meshes/calf.dae scale=1 1 1
- link lh_upperleg: geometry collision box size=0.25 0.0374 0.043; visual mesh filename=package://aliengo_description/meshes/thigh.dae scale=1 1 1
- link rf_hip: geometry collision cylinder length=0.0418 radius=0.046; visual mesh filename=package://aliengo_description/meshes/hip.dae scale=1 1 1
- link rf_lowerleg: geometry collision box size=0.25 0.0208 0.016; visual mesh filename=package://aliengo_description/meshes/calf.dae scale=1 1 1
- link rf_upperleg: geometry collision box size=0.25 0.0374 0.043; visual mesh filename=package://aliengo_description/meshes/thigh_mirror.dae scale=1 1 1
- link rh_hip: geometry collision cylinder length=0.0418 radius=0.046; visual mesh filename=package://aliengo_description/meshes/hip.dae scale=1 1 1
- link rh_lowerleg: geometry collision box size=0.25 0.0208 0.016; visual mesh filename=package://aliengo_description/meshes/calf.dae scale=1 1 1
- link rh_upperleg: geometry collision box size=0.25 0.0374 0.043; visual mesh filename=package://aliengo_description/meshes/thigh_mirror.dae scale=1 1 1
Joints:
- joint lf_hfe_joint: limit effort=44 velocity=20 -> lower=3.141592653589793 upper=-3.141592653589793 effort=44 velocity=20; type continuous -> revolute
- joint lh_hfe_joint: limit effort=44 velocity=20 -> lower=3.141592653589793 upper=-3.141592653589793 effort=44 velocity=20; type continuous -> revolute
- joint rf_hfe_joint: limit effort=44 velocity=20 -> lower=3.141592653589793 upper=-3.141592653589793 effort=44 velocity=20; type continuous -> revolute
- joint rh_hfe_joint: limit effort=44 velocity=20 -> lower=3.141592653589793 upper=-3.141592653589793 effort=44 velocity=20; type continuous -> revolute
