Commit message: Update a1 params

File: wolf_planner/config/a1/a1.urdf (robot description, URDF)
Before this commit: robot a1, 23 links, 22 joints
Links:
- link lf_hip: geometry collision cylinder length=0.04 radius=0.046; visual mesh filename=package://a1_description/meshes/hip.dae scale=1 1 1
- link lf_lowerleg: geometry collision box size=0.2 0.016 0.016; visual mesh filename=package://a1_description/meshes/calf.dae scale=1 1 1
- link lf_upperleg: geometry collision box size=0.2 0.0245 0.034; visual mesh filename=package://a1_description/meshes/thigh.dae scale=1 1 1
- link lh_hip: geometry collision cylinder length=0.04 radius=0.046; visual mesh filename=package://a1_description/meshes/hip.dae scale=1 1 1
- link lh_lowerleg: geometry collision box size=0.2 0.016 0.016; visual mesh filename=package://a1_description/meshes/calf.dae scale=1 1 1
- link lh_upperleg: geometry collision box size=0.2 0.0245 0.034; visual mesh filename=package://a1_description/meshes/thigh.dae scale=1 1 1
- link rf_hip: geometry collision cylinder length=0.04 radius=0.046; visual mesh filename=package://a1_description/meshes/hip.dae scale=1 1 1
- link rf_lowerleg: geometry collision box size=0.2 0.016 0.016; visual mesh filename=package://a1_description/meshes/calf.dae scale=1 1 1
- link rf_upperleg: geometry collision box size=0.2 0.0245 0.034; visual mesh filename=package://a1_description/meshes/thigh_mirror.dae scale=1 1 1
- link rh_hip: geometry collision cylinder length=0.04 radius=0.046; visual mesh filename=package://a1_description/meshes/hip.dae scale=1 1 1
- link rh_lowerleg: geometry collision box size=0.2 0.016 0.016; visual mesh filename=package://a1_description/meshes/calf.dae scale=1 1 1
- link rh_upperleg: geometry collision box size=0.2 0.0245 0.034; visual mesh filename=package://a1_description/meshes/thigh_mirror.dae scale=1 1 1
