Commit message: Rename trunk -> base_link for go1

File: wolf_planner/config/robots/go1/go1.urdf (robot description, URDF)
Before this commit: robot go1, 24 links, 23 joints
Links:
- removed link trunk
- added link base_link, mass 5.204; collision box size=0.3762 0.0935 0.114; visual mesh filename=package://go1_description/meshes/trunk.dae scale=1 1 1
Joints:
- joint floating_base_joint: child trunk -> base_link
- joint imu_joint: parent trunk -> base_link
- joint lf_haa_joint: parent trunk -> base_link
- joint lh_haa_joint: parent trunk -> base_link
- joint lidar_cage_to_lidar: parent trunk -> base_link
- joint rf_haa_joint: parent trunk -> base_link
- joint rh_haa_joint: parent trunk -> base_link
